File: KiCad/FlightLight_V2.0/FlightLight.kicad_pcb (KiCad board)
At the start: 2 copper layers, 33.5 x 35.5 mm, 26 parts, among them J3 Conn_02x05_Odd_Even, SW1 AP, U2 ULN2003, U3 ESP-12F, U4 AMS1117-3.3

Commit message: Add files via upload
Parts:
- added R11: 680k, Resistor_SMD:R_0805_2012Metric_Pad1.20x1.40mm_HandSolder, F.Cu at (106.5, 70.0)
- C2: value 100nF -> 100n; footprint Capacitor_SMD:C_0805_2012Metric_Pad1.18x1.45mm_HandSolder -> Capacitor_SMD:C_1206_3216Metric_Pad1.33x1.80mm_HandSolder
- C3, C4: footprint Capacitor_SMD:C_0805_2012Metric_Pad1.18x1.45mm_HandSolder -> Capacitor_SMD:C_1206_3216Metric_Pad1.33x1.80mm_HandSolder
- R10: value 1300k -> 680k
- R8: footprint Resistor_SMD:R_0805_2012Metric_Pad1.20x1.40mm_HandSolder -> Resistor_SMD:R_1206_3216Metric_Pad1.30x1.75mm_HandSolder
- moved R10 1.00 mm to (106.5, 72.0)
- moved C2 0.97 mm to (124.5, 76.4)
- moved R8 0.50 mm to (126.0, 85.5)
- moved R9 0.50 mm to (106.5, 74.0)
- moved C3 0.44 mm to (123.5, 85.4)
- moved C4 0.44 mm to (113.5, 85.4)
Connections:
- R10 pad 2: +BATT -> Net-(R10-Pad2)
Routing:
- net Net-(R10-Pad2): track 0.00 -> 2.00 mm
- net 3,3V: track 68.3 -> 66.5 mm
- net -BATT: track 6.15 -> 4.96 mm, vias 13 -> 14
- net D2: track 15.0 -> 14.0 mm
- net /CH2: track 11.0 -> 10.0 mm
- net ADC: track 12.2 -> 13.0 mm
Other:
- board text added: "sLiachdDingens"
- board text added: "sLiachdDingens V2"
- board text removed: "FlightLight V2"
- board text removed: "FlightLight V2.0"
