File: KiCad/FlightLight_V2.0/FlightLight.kicad_sch (KiCad schematic)
At the start: 26 parts, among them J3 Conn_02x05_Odd_Even, SW1 AP, U2 ULN2003, U3 ESP-12F, U4 AMS1117-3.3

Commit message: Add files via upload
Parts:
- added R11: 680k, Resistor_SMD:R_0805_2012Metric_Pad1.20x1.40mm_HandSolder, symbol Device:R
- C2: value 100nF -> 100n
- R10: value 1300k -> 680k
Connections:
- net +BATT: now also R11.2; no longer R10.2
- new net: R10.2, R11.1
Changed lines of the file:
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@@
 	(wire
 		(pts
-			(xy 160.02 107.95) (xy 160.02 127)
+			(xy 160.02 107.95) (xy 160.02 118.11)
 		)
 		(stroke
@@
 	(wire
 		(pts
+			(xy 160.02 125.73) (xy 160.02 127)
+		)
+		(stroke
+			(width 0)
+			(type default)
+		)
+	)
+	(wire
+		(pts
 			(xy 87.63 137.16) (xy 91.44 137.16)
 		)
@@
 			)
 		)
-		(property "Value" "100nF"
+		(property "Value" "100n"
 			(at 173.101 130.683 0)
 			(effects
@@
 	)
 	(symbol
+		(lib_id "Device:R")
+		(at 160.02 121.92 180)
+		(unit 1)
+		(exclude_from_sim no)
+		(in_bom yes)
+		(on_board yes)
+		(dnp no)
+		(property "Reference" "R11"
+			(at 158.242 123.0884 0)
+			(effects
+				(font
+					(size 1.27 1.27)
+				)
+				(justify left)
+			)
+		)
+		(property "Value" "680k"
+			(at 158.242 120.777 0)
+			(effects
+				(font
+					(size 1.27 1.27)
+				)
+				(justify left)
+			)
+		)
+		(property "Footprint" "Resistor_SMD:R_0805_2012Metric_Pad1.20x1.40mm_HandSolder"
+			(at 161.798 121.92 90)
+			(effects
+				(font
+					(size 1.27 1.27)
+				)
+				(hide yes)
+			)
+		)
+		(property "Datasheet" "~"
+			(at 160.02 121.92 0)
+			(effects
+				(font
+					(size 1.27 1.27)
+				)
+				(hide yes)
+			)
+		)
+		(property "Description" ""
+			(at 160.02 121.92 0)
+			(effects
+				(font
+					(size 1.27 1.27)
+				)
+				(hide yes)
+			)
+		)
+		(pin "2"
+		)
+		(pin "1"
+		)
+		(instances
+			(project "FlightLight"
+				(path "/1ec19e6d-0844-4ed7-9061-0a9fb2bcdc9b"
+					(reference "R11")
+					(unit 1)
+				)
+			)
+		)
+	)
+	(symbol
 		(lib_id "RF_Module:ESP-12F")
 		(at 210.82 68.58 0)
@@
 			)
 		)
-		(property "Value" "1300k"
+		(property "Value" "680k"
 			(at 158.242 129.667 0)
 			(effects
